File: layout/sensor_v0.2.sch (EAGLE design)
At the start: 25 parts, among them IC1 DS2406P, IC2 AZ1117-5.0, K1 833H-1C-C-12VDC, T1 BSS84, X1 1751264

Commit message: lamp 1w ds2423 emulator
Other:
- note removed: "org: 2k2 +3k3"
Changed lines of the file:
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@@
 <sheet>
 <plain>
-<text x="50.8" y="154.94" size="1.778" layer="91">org: 2k2 +3k3</text>
 <wire x1="114.3" y1="170.18" x2="114.3" y2="17.78" width="0.1524" layer="94" style="longdash"/>
 </plain>
